Commit message: added wwlambda model

File: Hector_ROS_Simulation/hector_description/xacro/gazebo.xacro (robot description, xacro)
@@ -106,4 +106,20 @@
         <material>Gazebo/Grey</material>
     </gazebo>
+    <gazebo reference="bumper_LF">
+        <mu1>3</mu1>
+        <mu2>3</mu2>
+        <kp  value="1000000.0"/>
+        <kd  value="1000.0"/>
+        <self_collide>0</self_collide>
+        <material>Gazebo/Red</material>
+    </gazebo>
+    <gazebo reference="bumper_LB">
+        <mu1>3</mu1>
+        <mu2>3</mu2>
+        <kp  value="1000000.0"/>
+        <kd  value="1000.0"/>
+        <self_collide>0</self_collide>
+        <material>Gazebo/Red</material>
+    </gazebo>
     <!--R leg -->
     <gazebo reference="R_hip">
@@ -145,3 +161,19 @@
         <material>Gazebo/Grey</material>
     </gazebo>
+    <gazebo reference="bumper_RF">
+        <mu1>3</mu1>
+        <mu2>3</mu2>
+        <kp  value="1000000.0"/>
+        <kd  value="1000.0"/>
+        <self_collide>0</self_collide>
+        <material>Gazebo/Red</material>
+    </gazebo>
+    <gazebo reference="bumper_RB">
+        <mu1>3</mu1>
+        <mu2>3</mu2>
+        <kp  value="1000000.0"/>
+        <kd  value="1000.0"/>
+        <self_collide>0</self_collide>
+        <material>Gazebo/Red</material>
+    </gazebo>
 </robot>

File: Hector_ROS_Simulation/hector_description/xacro/leg.xacro (robot description, xacro)
@@ -143,5 +143,5 @@
             <child link="${name}_thigh"/>
             <axis xyz="0 1 0"/>
-            <joint_properties damping="${damping}" friction="${friction}"/>
+            <dynamics damping="${damping}" friction="${friction}"/>
             <!-- <limit effort="${thigh_torque_max}" velocity="${thigh_velocity_max}"/> -->
             <limit effort="${thigh_torque_max}" velocity="${thigh_velocity_max}" lower="${thigh_min*PI/180.0}" upper="${thigh_max*PI/180.0}"/>
@@ -226,5 +226,5 @@
             <child link="${name}_calf"/>
             <axis xyz="0 1 0"/>
-            <joint_properties damping="${damping}" friction="${friction}"/>
+            <dynamics damping="${damping}" friction="${friction}"/>
             <limit effort="${calf_torque_max}" velocity="${calf_velocity_max}" lower="${calf_min*PI/180.0}" upper="${calf_max*PI/180.0}"/>
         </joint>
@@ -264,5 +264,5 @@
             <child link="${name}_toe"/>
             <axis xyz="0 1 0"/>
-            <joint_properties damping="${damping}" friction="${friction}"/>
+            <dynamics damping="${damping}" friction="${friction}"/>
             <limit effort="${toe_torque_max}" velocity="${toe_velocity_max}" lower="${toe_min*PI/180.0}" upper="${toe_max*PI/180.0}"/>
         </joint>
