Commit message: bear_actuator_ros update

File: Hector_ROS_Simulation/hector_description/xacro/wwlambda_const.xacro (robot description, xacro)
@@ -16,7 +16,10 @@
     <xacro:property name="toe_joint_max" value="1.75"/>
     <xacro:property name="toe_joint_min" value="-1.75"/>
-    <xacro:property name="thigh_angle" value="0.785398163"/>
-    <xacro:property name="calf_angle" value="-1.570796327"/>
-    <xacro:property name="toe_angle" value="0.785398163"/>
+    <!-- <xacro:property name="thigh_angle" value="0.785398163"/> -->
+    <!-- <xacro:property name="calf_angle" value="-1.570796327"/> -->
+    <!-- <xacro:property name="toe_angle" value="0.785398163"/> -->
+    <xacro:property name="thigh_angle" value="0.0"/>
+    <xacro:property name="calf_angle" value="0.0"/>
+    <xacro:property name="toe_angle" value="0.0"/>
     <!-- trunk value -->
     <!-- collision -->
