Commit message: dfm mode driver update

File: Hector_ROS_Simulation/hector_description/xacro/bear_dfm_test.urdf (robot description, URDF)
Before this commit: robot bear_dfm_test, 5 links, 4 joints
Links:
- link arm1: geometry visual box size=0.15 0.01 0.005
- link arm2: geometry visual box size=0.15 0.01 0.005
