Commit message: various minor corrections

File: Hector_ROS_Simulation/hector_description/xacro/bumper.xacro (robot description, xacro)
@@ -53,9 +53,9 @@
     </gazebo>
 </xacro:macro>
-<xacro:property name="bumper_width" value="0.030"/>
+<xacro:property name="bumper_width" value="0.040"/>
 <xacro:property name="bumper_height" value="0.002"/>
-<xacro:property name="bumper_depth" value="0.030"/>
+<xacro:property name="bumper_depth" value="0.040"/>
 <xacro:property name="collision_avoidance" value="0.001"/>
-<xacro:property name="t_height" value="0.029"/>
-<xacro:property name="t_depth" value="0.100"/>
+<xacro:property name="t_height" value="0.037"/>
+<xacro:property name="t_depth" value="0.120"/>
 </robot>

File: Hector_ROS_Simulation/hector_description/xacro/wwlambda_r2.xacro (robot description, xacro)
@@ -60,5 +60,5 @@
     <link name="body">
         <inertial>
-            <mass value="1.3"/>
+            <mass value="1.02"/>
             <origin rpy="0 0 0" xyz="0 0 0"/>
             <inertia ixx="3035947e-9" ixy="-1669e-9" ixz="2793e-9" iyy="2992228e-9" iyz="17720e-9" izz="3906372e-9"/>
@@ -259,12 +259,12 @@
             <origin rpy="0 0 0" xyz="0 0 0"/>
             <geometry>
-                <mesh filename="package://hector_description/meshes/wwlambda/ww_lambda_left_foot.stl" scale="1 1 1 "/>
+                <mesh filename="package://hector_description/meshes/wwlambda/foot.stl" scale="1 1 1 "/>
             </geometry>
             <material name="green"/>
         </visual>
         <collision>
-            <origin rpy="0 0 0" xyz="0 0 -0.023"/>
-            <geometry>
-                <box size="0.100 0.030 0.012"/>
+            <origin rpy="0 0 0" xyz="0 0 -0.0265"/>
+            <geometry>
+                <box size="0.120 0.040 0.021"/>
             </geometry>
         </collision>
@@ -410,12 +410,12 @@
             <origin rpy="0 0 0" xyz="0 0 0"/>
             <geometry>
-                <mesh filename="package://hector_description/meshes/wwlambda/ww_lambda_right_foot.stl" scale="1 1 1"/>
+                <mesh filename="package://hector_description/meshes/wwlambda/foot.stl" scale="1 1 1"/>
             </geometry>
             <material name="green"/>
         </visual>
         <collision>
-            <origin rpy="0 0 0" xyz="0 0 -0.023"/>
-            <geometry>
-                <box size="0.100 0.030 0.012"/>
+            <origin rpy="0 0 0" xyz="0 0 -0.0265"/>
+            <geometry>
+                <box size="0.120 0.040 0.021"/>
             </geometry>
         </collision>
